File: KiCad/espScale/espScale.kicad_pcb (KiCad board)
At the start: 2 copper layers, 46.4 x 71.1 mm, 1 part, among them U1 NodeMCU1.0(ESP-12E)

Commit message: pcb
Parts:
- added J1: 2-pin_power_input_header, My_Headers:2-pin_power_input_header_larger_pads, F.Cu at (108.0, 101.6)
- added U6: HX711_Load_Cell_Amplifier, My_Parts:HX711 Load Cell Amplifier w_pinsockets_large, F.Cu at (114.9, 68.6)
Connections:
- U1 pad 22: unconnected-(U1-Pad22) -> SCK
Routing:
- net SCK: track 0.00 -> 78.6 mm
- net DT: track 0.00 -> 62.7 mm
- net +5V: track 0.00 -> 32.6 mm
- net GND: track 0.00 -> 31.7 mm
Other:
- board size 46.4 x 71.1 mm -> 53.3 x 59.7 mm

Commit message: kicad
Parts:
- added U2: 3-wire_Load_Cell, My_Headers:3-pin_load_cell_header_large, F.Cu at (92.1, 73.0)
- added U3: ~, My_Headers:3-pin_load_cell_header_large, F.Cu at (92.1, 109.2)
- added U4: 3-wire_Load_Cell, My_Headers:3-pin_load_cell_header_large, F.Cu at (92.1, 97.2)
- added U5: ~, My_Headers:3-pin_load_cell_header_large, F.Cu at (92.1, 85.1)
- J1: footprint My_Headers:2-pin_power_input_header_larger_pads -> My_Headers:2-pin_power_input_header
- moved U1 25.0 mm to (127.0, 74.9)
- moved U6 16.9 mm to (119.4, 84.9)
- moved J1 16.6 mm to (106.7, 118.1), turned to 0 degrees
Connections:
- U6 pad 3: (no net) -> Net-(U6-Pad3)
Routing:
- net Net-(U3-Pad1): track 0.00 -> 218.3 mm
- net Net-(U2-Pad3): track 0.00 -> 187.5 mm
- net Net-(U3-Pad2): track 0.00 -> 33.1 mm
- net Net-(U2-Pad2): track 0.00 -> 30.9 mm
- net Net-(U2-Pad1): track 0.00 -> 30.4 mm, vias 0 -> 2
- net Net-(U6-Pad3): track 0.00 -> 28.2 mm
- net Net-(U5-Pad2): track 0.00 -> 26.9 mm
- net SCK: track 78.6 -> 100.2 mm
- net Net-(U4-Pad3): track 0.00 -> 20.7 mm, vias 0 -> 2
- net DT: track 62.7 -> 78.8 mm
- net GND: track 31.7 -> 44.5 mm
- net +5V: track 32.6 -> 30.6 mm
- added copper zone on B.Cu, net (none)
- added copper zone on B.Cu, net GND
Other:
- board size 53.3 x 59.7 mm -> 73.7 x 64.1 mm
- board text added: "espScale Design: Jon Sagebrand github.com/jonsag"

Commit message: kicad page settings
Parts:
- U2, U3, U4, U5: footprint My_Headers:3-pin_load_cell_header_large -> My_Headers:3-pin JST load cell
- moved U5 0.67 mm to (92.8, 85.2), turned to 0 degrees
- moved U2 0.12 mm to (92.1, 73.1), turned to 0 degrees
- moved U3 0.11 mm to (92.1, 109.3), turned to 0 degrees
- moved U4 0.11 mm to (92.1, 97.3), turned to 0 degrees
Other:
- board text added: "${TITLE}-${REVISION} Design: Jon Sagebrand github.com/jonsag"
- board text removed: "espScale Design: Jon Sagebrand github.com/jonsag"

Commit message: new PCB, added 3-pin LCD
Parts:
- added H1: MountingHole, MountingHole:MountingHole_3.2mm_M3, F.Cu at (163.8, 66.0)
- added H2: MountingHole, MountingHole:MountingHole_3.2mm_M3, F.Cu at (90.8, 119.4)
- added H3: MountingHole, MountingHole:MountingHole_3.2mm_M3, F.Cu at (163.8, 119.4)
- added H4: MountingHole, MountingHole:MountingHole_3.2mm_M3, F.Cu at (90.8, 66.0)
- added J2: 5-pin_LCD, My_Headers:5-pin JST LiquidCrystal595, F.Cu at (164.2, 101.0)
- added J3: I2C Display, My_Headers:4-pin JST LCD, F.Cu at (163.2, 93.3)
- added SW1: Reset, My_Misc:SW_PUSH_6mm_large, F.Cu at (160.7, 79.4)
- renumbered U2 to U1, U3 to U2, U4 to U3, U5 to U4, U6 to U5, U1 to U6
Connections:
- U6 pad 10: unconnected-(U1-Pad10) -> GND
- U6 pad 17: unconnected-(U1-Pad17) -> GND
- U6 pad 20: unconnected-(U1-Pad20) -> Clock
- U6 pad 21: unconnected-(U1-Pad21) -> Latch
- U6 pad 24: unconnected-(U1-Pad24) -> GND
- U6 pad 26: unconnected-(U1-Pad26) -> Net-(U6-Pad26)
- U6 pad 27: unconnected-(U1-Pad27) -> Data
- U6 pad 28: unconnected-(U1-Pad28) -> SDA
- U6 pad 29: unconnected-(U1-Pad29) -> SCL
Routing:
- net Net-(U2-Pad1): track 218.3 -> 26.1 mm
- net GND: track 44.5 -> 198.2 mm
- net Net-(U1-Pad3): track 187.5 -> 57.4 mm
- net +5V: track 30.6 -> 114.0 mm, vias 0 -> 2
- net Net-(U6-Pad26): track 0.00 -> 26.7 mm
- net Data: track 0.00 -> 23.6 mm
- net SDA: track 0.00 -> 12.6 mm
- net SCL: track 0.00 -> 12.5 mm
- net Latch: track 0.00 -> 11.4 mm
- net Clock: track 0.00 -> 11.4 mm
- net SCK: track 100.2 -> 92.8 mm
- net DT: track 78.8 -> 81.2 mm
Other:
- board size 73.7 x 64.1 mm -> 81.9 x 62.2 mm
- board text added: "1"
- board text added: "2"
- board text added: "3"
