File: KiCad/espScale/espScale.kicad_sch (KiCad schematic)
At the start: 6 parts, among them U1 NodeMCU1.0(ESP-12E), U2 3-wire_Load_Cell, U4 3-wire_Load_Cell, U6 HX711_Load_Cell_Amplifier

Commit message: pcb
Parts:
- added J1: (no value), symbol My_Headers:2-pin_power_input_header
Connections:
- net +5V: now also J1.1 (VCC)
- net GND: now also J1.2 (GND)
Changed lines of the file:
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@@
+    (stroke (width 0) (type default) (color 0 0 0 0))
+  )
+  (wire (pts (xy 91.44 55.88) (xy 91.44 60.96))
     (stroke (width 0) (type default) (color 0 0 0 0))
   )
@@
     (stroke (width 0) (type default) (color 0 0 0 0))
   )
+  (wire (pts (xy 88.9 55.88) (xy 91.44 55.88))
+    (stroke (width 0) (type default) (color 0 0 0 0))
+  )
   (wire (pts (xy 97.79 118.11) (xy 129.54 118.11))
     (stroke (width 0) (type default) (color 0 0 0 0))
@@
     (stroke (width 0) (type default) (color 0 0 0 0))
   )
+  (wire (pts (xy 88.9 53.34) (xy 91.44 53.34))
+    (stroke (width 0) (type default) (color 0 0 0 0))
+  )
   (wire (pts (xy 102.87 148.59) (xy 97.79 148.59))
     (stroke (width 0) (type default) (color 0 0 0 0))
@@
   )
   (wire (pts (xy 184.15 142.24) (xy 184.15 123.19))
+    (stroke (width 0) (type default) (color 0 0 0 0))
+  )
+  (wire (pts (xy 91.44 53.34) (xy 91.44 48.26))
     (stroke (width 0) (type default) (color 0 0 0 0))
   )
@@
     (pin "9")
   )
+  (symbol (lib_id "power:+5V") (at 91.44 48.26 0) (unit 1)
+    (in_bom yes) (on_board yes) (fields_autoplaced)
+    (property "Reference" "#PWR0105" (id 0) (at 91.44 52.07 0)
+      (effects (font (size 1.27 1.27)) hide)
+    )
+    (property "Value" "" (id 1) (at 91.44 44.6842 0))
+    (property "Footprint" "" (id 2) (at 91.44 48.26 0)
+      (effects (font (size 1.27 1.27)) hide)
+    )
+    (property "Datasheet" "" (id 3) (at 91.44 48.26 0)
+      (effects (font (size 1.27 1.27)) hide)
+    )
+    (pin "1")
+  )
   (symbol (lib_id "power:+5V") (at 137.16 30.48 0) (unit 1)
     (in_bom yes) (on_board yes) (fields_autoplaced)
@@
     (pin "1")
   )
+  (symbol (lib_id "power:GND") (at 91.44 60.96 0) (unit 1)
+    (in_bom yes) (on_board yes) (fields_autoplaced)
+    (property "Reference" "#PWR0106" (id 0) (at 91.44 67.31 0)
+      (effects (font (size 1.27 1.27)) hide)
+    )
+    (property "Value" "" (id 1) (at 91.44 65.4034 0))
+    (property "Footprint" "" (id 2) (at 91.44 60.96 0)
+      (effects (font (size 1.27 1.27)) hide)
+    )
+    (property "Datasheet" "" (id 3) (at 91.44 60.96 0)
+      (effects (font (size 1.27 1.27)) hide)
+    )
+    (pin "1")
+  )
   (symbol (lib_name "3-wire_Load_Cell_2") (lib_id "My_Parts:3-wire_Load_Cell") (at 97.79 118.11 0) (mirror y) (unit 1)
     (in_bom yes) (on_board yes) (fields_autoplaced)
@@
     (pin "3")
   )
+  (symbol (lib_id "My_Headers:2-pin_power_input_header") (at 83.82 53.34 0) (mirror y) (unit 1)
+    (in_bom yes) (on_board yes) (fields_autoplaced)
+    (property "Reference" "J1" (id 0) (at 84.455 51.72 0))
+    (property "Value" "" (id 1) (at 83.82 58.42 0)
+      (effects (font (size 1.27 1.27)) hide)
+    )
+    (property "Footprint" "" (id 2) (at 82.55 60.96 0)
+      (effects (font (size 1.27 1.27)) hide)
+    )
+    (property "Datasheet" "~" (id 3) (at 83.82 53.34 0)
+      (effects (font (size 1.27 1.27)) hide)
+    )
+    (pin "1")
+    (pin "2")
+  )
   (symbol (lib_id "My_Parts:3-wire_Load_Cell") (at 129.54 118.11 0) (unit 1)
     (in_bom yes) (on_board yes) (fields_autoplaced)
@@
       (reference "#PWR0104") (unit 1) (value "GND") (footprint "")
     )
+    (path "/3896d8e3-13c4-4e01-a766-927ff0202f2b"
+      (reference "#PWR0105") (unit 1) (value "+5V") (footprint "")
+    )
+    (path "/5b40dd14-548e-441a-8e60-aabed75d2537"
+      (reference "#PWR0106") (unit 1) (value "GND") (footprint "")
+    )
+    (path "/9b5bbbea-ca45-4da3-962b-10accf46ad7c"
+      (reference "J1") (unit 1) (value "2-pin_power_input_header") (footprint "My_Headers:2-pin_power_input_header_larger_pads")
+    )
     (path "/32f4eb0d-8b7c-4e0f-8b4a-904219172497"
       (reference "U1") (unit 1) (value "NodeMCU1.0(ESP-12E)") (footprint "My_ESP8266:NodeMCU-LoLinV3_w_pinsockets_large")
@@
     )
     (path "/3c667cba-91d1-4464-8b34-8c6b7fcac30a"
-      (reference "U6") (unit 1) (value "HX711_Load_Cell_Amplifier") (footprint "")
-    )
-  )
+      (reference "U6") (unit 1) (value "HX711_Load_Cell_Amplifier") (footprint "My_Parts:HX711 Load Cell Amplifier w_pinsockets_large")
+    )
+  )

Commit message: kicad
Parts:
- J1: value (none) -> 2-pin_power_input_header; footprint (none) -> My_Headers:2-pin_power_input_header
- U2, U3, U4, U5: footprint (none) -> My_Headers:3-pin_load_cell_header_large
- U6: footprint (none) -> My_Parts:HX711 Load Cell Amplifier w_pinsockets_large
Connections:
- net at U4.2 (Red): now also U6.3 (A-); no longer U6.4 (A-)
Other:
- moved on the sheet: U2, U3, U4, U5, U6

Commit message: kicad page settings
Parts:
- U2, U3, U4, U5: footprint My_Headers:3-pin_load_cell_header_large -> My_Headers:3-pin JST load cell
Other:
- title: (none) -> espScale
Changed lines of the file:
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@@
 (kicad_sch (version 20211123) (generator eeschema)
   (paper "A4")
+  (title_block
+    (title "espScale")
+    (date "2022-09-18")
+    (rev "0.1")
+  )
   (wire (pts (xy 184.15 127) (xy 189.23 127))
     (stroke (width 0) (type default) (color 0 0 0 0))
@@
       (effects (font (size 1.27 1.27)) (justify left))
     )
-    (property "Footprint" "My_Headers:3-pin_load_cell_header_large" (id 2) (at 139.319 124.841 0)
+    (property "Footprint" "My_Headers:3-pin JST load cell" (id 2) (at 139.319 124.841 0)
       (effects (font (size 1.27 1.27)) hide)
     )
@@
     (property "Reference" "U2" (id 0) (at 95.25 97.316 0))
     (property "Value" "3-wire_Load_Cell" (id 1) (at 95.25 99.8529 0))
-    (property "Footprint" "My_Headers:3-pin_load_cell_header_large" (id 2) (at 98.171 99.441 0)
+    (property "Footprint" "My_Headers:3-pin JST load cell" (id 2) (at 98.171 99.441 0)
       (effects (font (size 1.27 1.27)) hide)
     )
@@
       (effects (font (size 1.27 1.27)) (justify left))
     )
-    (property "Footprint" "My_Headers:3-pin_load_cell_header_large" (id 2) (at 139.319 99.441 0)
+    (property "Footprint" "My_Headers:3-pin JST load cell" (id 2) (at 139.319 99.441 0)
       (effects (font (size 1.27 1.27)) hide)
     )
@@
     (property "Reference" "U3" (id 0) (at 95.25 122.716 0))
     (property "Value" "~" (id 1) (at 95.25 125.2529 0))
-    (property "Footprint" "My_Headers:3-pin_load_cell_header_large" (id 2) (at 98.171 124.841 0)
+    (property "Footprint" "My_Headers:3-pin JST load cell" (id 2) (at 98.171 124.841 0)
       (effects (font (size 1.27 1.27)) hide)
     )
@@
     )
     (path "/8af7217e-6b6b-49c7-a1b8-be8a38ecb040"
-      (reference "U2") (unit 1) (value "3-wire_Load_Cell") (footprint "My_Headers:3-pin_load_cell_header_large")
+      (reference "U2") (unit 1) (value "3-wire_Load_Cell") (footprint "My_Headers:3-pin JST load cell")
     )
     (path "/d6d827e1-8037-4a64-9433-b930cfff7250"
-      (reference "U3") (unit 1) (value "~") (footprint "My_Headers:3-pin_load_cell_header_large")
+      (reference "U3") (unit 1) (value "~") (footprint "My_Headers:3-pin JST load cell")
     )
     (path "/bad23df6-f465-434f-8740-c4824bad6534"
-      (reference "U4") (unit 1) (value "3-wire_Load_Cell") (footprint "My_Headers:3-pin_load_cell_header_large")
+      (reference "U4") (unit 1) (value "3-wire_Load_Cell") (footprint "My_Headers:3-pin JST load cell")
     )
     (path "/3209d3a7-a6c2-49ab-93de-4f7ab80f7cda"
-      (reference "U5") (unit 1) (value "~") (footprint "My_Headers:3-pin_load_cell_header_large")
+      (reference "U5") (unit 1) (value "~") (footprint "My_Headers:3-pin JST load cell")
     )
     (path "/3c667cba-91d1-4464-8b34-8c6b7fcac30a"

Commit message: new PCB, added 3-pin LCD
Parts:
- added H1, H2, H3, H4: MountingHole, MountingHole:MountingHole_3.2mm_M3, symbol Mechanical:MountingHole
- added J2: 5-pin_LCD, My_Headers:5-pin JST LiquidCrystal595, symbol My_Headers:5-pin_LCD
- added J3: I2C Display, My_Headers:4-pin JST LCD, symbol My_Headers:4-pin_I2C_LCD_header
- added SW1: Reset, My_Misc:SW_PUSH_6mm_large, symbol Switch:SW_Push
- renumbered U2 to U1, U3 to U2, U4 to U3, U5 to U4, U6 to U5, U1 to U6
Connections:
- net +5V: now also J2.4 (+5V), J3.1 (+5V)
- net GND: now also U6.10 (GND), U6.17 (GND), U6.24 (GND), J2.5 (GND), J3.2 (GND), SW1.2
- net Clock: now reaches U6.20 (D8(GPIO15))
- net Clock: now also J2.3 (Clock)
- net Latch: now reaches U6.21 (D7(GPIO13))
- net Latch: now also J2.2 (Latch)
- net at U6.26 (D4(GPIO2)): now also SW1.1
- net Data: now reaches U6.27 (D3(GPIO0))
- net Data: now also J2.1 (Data)
- net SDA: now reaches U6.28 (D2(GPIO4))
- net SDA: now also J3.3 (SDA)
- net SCL: now reaches U6.29 (D1(GPIO5))
- net SCL: now also J3.4 (SCL)
